Commit message: Started work on the data collection environment.  Note: I decided to use a shorter peg and a shorter box to see if that improved results

File: data/objects/homemade_objects/peg.urdf (robot description, URDF)
Before this commit: robot peg, 1 links, 0 joints
Links:
- link base_link: mass 1 -> 1.2
