Commit message: Further building out of data_collection environment.  Used a new strategy for placing the peg.

File: data/robot/rethink/sawyer_description/urdf/sawyer_arm_wsg50.urdf (robot description, URDF)
Before this commit: robot sawyer_no_base, 16 links, 15 joints
Links:
- added link focus_point; visual box size=0.002 0.002 0.002
Joints:
- added joint focus_point_joint: type fixed, parent gripper_base_link, child focus_point, origin xyz=0.0 0.0 0.1 rpy=0.0 0.0 0.0
